File: KiCad/custom locker/custom locker/custom locker.kicad_pcb (KiCad board)
At the start: 2 copper layers, 92 x 76 mm, 15 parts, among them J1 Servo Motor Connector, J2 Power, J3 HX711 load cell, J4 Hall Effect Sensor, U1 ESP32-DEVKITC-32D, U2 DM-OLED096-636

Commit message: final submission files
Connections:
- LS1 pad P: Net-(U1-IO32) -> Net-(U1-IO5)
- U1 pad J2-7: Net-(U1-IO32) -> unconnected-(U1-IO32-PadJ2-7)
- U1 pad J3-10: unconnected-(U1-IO5-PadJ3-10) -> Net-(U1-IO5)
Routing:
- net Net-(U1-IO32): track 55.1 -> 0.00 mm, vias 2 -> 0
- net Net-(U1-IO5): track 0.00 -> 28.0 mm, vias 0 -> 2
Other:
- board text added: "+5V"
- board text added: "CLOCK"
- board text added: "DATA"
- board text added: "GND"
- board text added: "IN"
- board text added: "SIGNAL"
