File: KiCad/custom locker/custom locker/custom locker.kicad_sch (KiCad schematic)
At the start: 8 parts, among them J1 servo motor connector, J3 HX711 load cell, SW1 SW_Push, SW2 SW_Push, SW3 SW_Push, U1 ESP32-DEVKITC-32D, U2 DM-OLED096-636

Commit message: finished pcb
Parts:
- added DOWN1: SW_Push, Button_Switch_Keyboard:SW_Cherry_MX_1.00u_PCB, symbol Switch:SW_Push
- added J2: Power, Connector_PinHeader_2.54mm:PinHeader_1x02_P2.54mm_Vertical, symbol Connector_Generic:Conn_01x02
- added J4: Hall Effect Sensor, Connector_PinHeader_2.54mm:PinHeader_1x03_P2.54mm_Vertical, symbol Connector_Generic:Conn_01x03
- J1: value servo motor connector -> Servo Motor Connector
- renumbered SW3 to CANCEL1, SW2 to SELECT1, SW1 to UP1
Connections:
- net +5V: now also J2.1 (Pin_1), J4.1 (Pin_1)
- net GND: now also DOWN1.1, J2.2 (Pin_2), J4.2 (Pin_2)
- net at U1.J2-5 (IO34): now also J4.3 (Pin_3)
- net SW4: now reaches U1.J3-12 (IO16)
- net SW4: now also DOWN1.2
Other:
- moved on the sheet: LS1

Commit message: little changes on PCB
mainly added screw holes
Parts:
- added H1, H2, H3, H4: MountingHole, MountingHole:MountingHole_4.3mm_M4, symbol Mechanical:MountingHole
Connections:
- net at J4.3 (Pin_3): now also U1.J2-8 (IO33); no longer U1.J2-5 (IO34)
Other:
- moved on the sheet: J4, LS1

Commit message: final submission files
Connections:
- net at U1.J2-7 (IO32): no longer LS1.P
- net at U1.J3-10 (IO5): now also LS1.P
Other:
- moved on the sheet: U2
